File: ortho-normal-keycaps/ortho-normal-keycap.kicad_pcb (KiCad board)
At the start: 2 copper layers, 68 parts, among them SW1 Switch, SW10 Switch, SW11 Switch, SW12 Switch, SW13 Switch, SW14 Switch, SW15 Switch, SW16 Switch, SW17 Switch, SW18 Switch, SW19 Switch, SW2 Switch, SW20 Switch, SW21 Switch, SW22 Switch, SW23 Switch, SW24 Switch, SW25 Switch, SW26 Switch, SW27 Switch, SW28 Switch, SW29 Switch, SW3 Switch, SW30 Switch, SW31 Switch, SW32 Switch, SW33 Switch, SW34 Switch, SW4 Switch, SW5 Switch, SW6 Switch, SW7 Switch, SW8 Switch, SW9 Switch, U1 nRF52840_E73-2G4M08S1C

Commit message: update project
Parts:
- removed SW34: Switch, eaglevlib-mx:SW_MX_1u
- added S1: MX_stab, eaglevlib-mx:STAB_MX_2.25u, F.Cu at (154.8, 114.3)
- added S2: MX_stab, eaglevlib-mx:STAB_MX_2.75u, F.Cu at (64.3, 95.2)
- D1, D10, D11, D12, D13, D14, D15, D16, D17, D18, D19, D2, D20, D21, D22, D23, D24, D25, D26, D27, D28, D29, D3, D30, D31, D32, D33, D4, D5, D6, D7, D8, D9, U1: moved to B.Cu
- SW16: footprint eaglevlib-mx:SW_MX_1u -> eaglevlib-mx:SW_MX_CapsLock
- SW30, SW31, SW32: footprint eaglevlib-mx:SW_MX_1u -> eaglevlib-mx:SW_MX_1.25u
- SW9: footprint eaglevlib-mx:SW_MX_1u -> eaglevlib-mx:SW_MX_1.5u
- moved SW7 155.3 mm to (171.4, 38.1)
- moved SW14 131.7 mm to (171.4, 57.1)
- moved SW6 131.1 mm to (152.4, 38.1)
- moved D29 113.7 mm to (52.7, 117.3), turned to 90 degrees
- moved SW21 108.4 mm to (171.4, 76.2)
- moved SW13 107.5 mm to (152.4, 57.1)
- moved SW5 106.8 mm to (133.3, 38.1)
- moved D22 106.4 mm to (38.4, 98.3), turned to 90 degrees
- moved U1 97.3 mm to (40.3, 37.5), turned to 180 degrees
- moved D30 95.9 mm to (74.1, 117.3), turned to 90 degrees
- moved SW29 93.4 mm to (47.6, 114.3)
- moved SW28 85.7 mm to (171.4, 95.2)
- moved SW20 84.3 mm to (152.4, 76.2)
- moved SW12 83.2 mm to (133.3, 57.1)
- moved D15 82.7 mm to (47.9, 79.2), turned to 90 degrees
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Routing:
- net Row 3: track 0.00 -> 138.1 mm
- net Row 2: track 0.00 -> 128.6 mm
- net Row 1: track 0.00 -> 123.8 mm
- net Row 0: track 0.00 -> 114.3 mm
- net Row 4: track 0.00 -> 107.2 mm
- net Col 1: track 0.00 -> 94.3 mm
- net Col 0: track 0.00 -> 93.9 mm
- net Col 2: track 0.00 -> 77.3 mm
- net Col 3: track 0.00 -> 77.2 mm
- net Col 5: track 0.00 -> 77.2 mm
- net Col 6: track 0.00 -> 57.1 mm
- net Col 4: track 0.00 -> 57.1 mm
- net Net-(D16-A): track 0.00 -> 10.7 mm
- net Net-(D33-A): track 0.00 -> 7.86 mm
- net Net-(D12-A): track 0.00 -> 7.86 mm
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
Commit message: replace nRF52840 with nice!nano
Parts:
- removed U1: nRF52840_E73-2G4M08S1C, PCM_marbastlib-various:nRF52840_E73-2G4M08S1C
- added U2: nice_nano, PCM_marbastlib-xp-promicroish:nice_nano_AH_USBup, F.Cu at (114.3, 47.6)
- S23: renamed from S2; value MX_stab -> S2
- S33: renamed from S1; value MX_stab -> S1
- moved D23 2.93 mm to (66.9, 99.9)
- moved D24 2.93 mm to (97.9, 99.9)
- moved D25 2.93 mm to (116.9, 99.9)
- moved D26 2.93 mm to (136.0, 99.9)
- moved D27 2.93 mm to (155.0, 99.9)
- moved D28 2.93 mm to (174.1, 99.9)
- moved D29 2.93 mm to (50.3, 119.0)
- moved D30 2.93 mm to (71.7, 119.0)
- moved D31 2.93 mm to (95.5, 119.0)
- moved D32 2.93 mm to (119.3, 119.0)
- moved D33 2.93 mm to (157.4, 119.0)
- moved D10 2.93 mm to (97.9, 61.8)
- moved D11 2.93 mm to (116.9, 61.8)
- moved D12 2.93 mm to (136.0, 61.8)
- moved D13 2.93 mm to (155.0, 61.8)
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Routing:
- net Col 1: track 94.3 -> 0.00 mm
- net Col 0: track 93.9 -> 0.00 mm
- net Col 2: track 77.3 -> 0.00 mm
- net Col 3: track 77.2 -> 0.00 mm
- net Col 5: track 77.2 -> 0.00 mm
- net Col 6: track 57.1 -> 0.00 mm
- net Col 4: track 57.1 -> 0.00 mm
- net Net-(D17-A): track 7.70 -> 16.0 mm
- net Net-(D24-A): track 7.86 -> 16.0 mm
- net Net-(D8-A): track 7.86 -> 0.00 mm
- net Row 4: track 107.2 -> 109.3 mm
- net Row 3: track 138.1 -> 138.8 mm
