File: ortho-normal-keycaps/ortho-normal-keycap.kicad_sch (KiCad schematic)
At the start: 68 parts, among them SW1 Switch, SW10 Switch, SW11 Switch, SW12 Switch, SW13 Switch, SW14 Switch, SW15 Switch, SW16 Switch, SW17 Switch, SW18 Switch, SW19 Switch, SW2 Switch, SW20 Switch, SW21 Switch, SW22 Switch, SW23 Switch, SW24 Switch, SW25 Switch, SW26 Switch, SW27 Switch, SW28 Switch, SW29 Switch, SW3 Switch, SW30 Switch, SW31 Switch, SW32 Switch, SW33 Switch, SW34 Switch, SW4 Switch, SW5 Switch, SW6 Switch, SW7 Switch, SW8 Switch, SW9 Switch, U1 nRF52840_E73-2G4M08S1C

Commit message: update project
Parts:
- removed SW34: Switch, eaglevlib-mx:SW_MX_1u, symbol ScottoKeebs:Placeholder_Keyswitch
- added S1: MX_stab, eaglevlib-mx:STAB_MX_2.25u, symbol PCM_marbastlib-mx:MX_stab
- added S2: MX_stab, eaglevlib-mx:STAB_MX_2.75u, symbol PCM_marbastlib-mx:MX_stab
- SW16: footprint eaglevlib-mx:SW_MX_1u -> eaglevlib-mx:SW_MX_CapsLock
- SW30, SW31, SW32: footprint eaglevlib-mx:SW_MX_1u -> eaglevlib-mx:SW_MX_1.25u
- SW9: footprint eaglevlib-mx:SW_MX_1u -> eaglevlib-mx:SW_MX_1.5u
Changed lines of the file:
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@@
 	)
 	(junction
-		(at 187.96 101.6)
-		(diameter 0)
-		(color 0 0 0 0)
-	)
-	(junction
 		(at 223.52 78.74)
 		(diameter 0)
@@
 	)
 	(symbol
+		(lib_id "PCM_marbastlib-mx:MX_stab")
+		(at 158.75 154.94 0)
+		(unit 1)
+		(exclude_from_sim no)
+		(in_bom yes)
+		(on_board yes)
+		(dnp no)
+		(fields_autoplaced yes)
+		(property "Reference" "S1"
+			(at 165.1 153.5429 0)
+			(effects
+				(font
+					(size 1.27 1.27)
+				)
+				(justify left)
+			)
+		)
+		(property "Value" "MX_stab"
+			(at 165.1 156.0829 0)
+			(effects
+				(font
+					(size 1.27 1.27)
+				)
+				(justify left)
+			)
+		)
+		(property "Footprint" "eaglevlib-mx:STAB_MX_2.25u"
+			(at 158.75 154.94 0)
+			(effects
+				(font
+					(size 1.27 1.27)
+				)
+				(hide yes)
+			)
+		)
+		(property "Datasheet" ""
+			(at 158.75 154.94 0)
+			(effects
+				(font
+					(size 1.27 1.27)
+				)
+				(hide yes)
+			)
+		)
+		(property "Description" "Cherry MX-style stabilizer"
+			(at 158.75 154.94 0)
+			(effects
+				(font
+					(size 1.27 1.27)
+				)
+				(hide yes)
+			)
+		)
+		(instances
+			(project ""
+				(path "/75ca063f-3e3a-4a56-b625-1bf464e147b8"
+					(reference "S1")
+					(unit 1)
+				)
+			)
+		)
+	)
+	(symbol
 		(lib_id "ScottoKeebs:Placeholder_Diode")
 		(at 228.6 68.58 90)
@@
 			)
 		)
-		(property "Footprint" "eaglevlib-mx:SW_MX_1u"
+		(property "Footprint" "eaglevlib-mx:SW_MX_1.25u"
 			(at 185.42 134.62 0)
 			(effects
@@
 			)
 		)
-		(property "Footprint" "eaglevlib-mx:SW_MX_1u"
+		(property "Footprint" "eaglevlib-mx:SW_MX_1.25u"
 			(at 205.74 134.62 0)
 			(effects
@@
 	)
 	(symbol
+		(lib_id "PCM_marbastlib-mx:MX_stab")
+		(at 181.61 154.94 0)
+		(unit 1)
+		(exclude_from_sim no)
+		(in_bom yes)
+		(on_board yes)
+		(dnp no)
+		(fields_autoplaced yes)
+		(property "Reference" "S2"
+			(at 187.96 153.5429 0)
+			(effects
+				(font
+					(size 1.27 1.27)
+				)
+				(justify left)
+			)
+		)
+		(property "Value" "MX_stab"
+			(at 187.96 156.0829 0)
+			(effects
+				(font
+					(size 1.27 1.27)
+				)
+				(justify left)
+			)
+		)
+		(property "Footprint" "eaglevlib-mx:STAB_MX_2.75u"
+			(at 181.61 154.94 0)
+			(effects
+				(font
+					(size 1.27 1.27)
+				)
+				(hide yes)
+			)
+		)
+		(property "Datasheet" ""
+			(at 181.61 154.94 0)
+			(effects
+				(font
+					(size 1.27 1.27)
+				)
+				(hide yes)
+			)
+		)
+		(property "Description" "Cherry MX-style stabilizer"
+			(at 181.61 154.94 0)
+			(effects
+				(font
+					(size 1.27 1.27)
+				)
+				(hide yes)
+			)
+		)
+		(instances
+			(project "ortho-normal-keycap"
+				(path "/75ca063f-3e3a-4a56-b625-1bf464e147b8"
+					(reference "S2")
+					(unit 1)
+				)
+			)
+		)
+	)
+	(symbol
 		(lib_id "ScottoKeebs:Placeholder_Keyswitch")
 		(at 215.9 115.57 0)
@@
 	(symbol
 		(lib_id "ScottoKeebs:Placeholder_Keyswitch")
-		(at 185.42 99.06 0)
-		(unit 1)
-		(exclude_from_sim no)
-		(in_bom yes)
-		(on_board yes)
-		(dnp no)
-		(fields_autoplaced yes)
-		(property "Reference" "SW34"
-			(at 185.42 91.44 0)
-			(effects
-				(font
-					(size 1.27 1.27)
-				)
-			)
-		)
-		(property "Value" "Switch"
-			(at 185.42 93.98 0)
-			(effects
-				(font
-					(size 1.27 1.27)
-				)
-			)
-		)
-		(property "Footprint" "eaglevlib-mx:SW_MX_1u"
-			(at 185.42 99.06 0)
-			(effects
-				(font
-					(size 1.27 1.27)
-				)
-				(hide yes)
-			)
-		)
-		(property "Datasheet" "~"
-			(at 185.42 99.06 0)
-			(effects
-				(font
-					(size 1.27 1.27)
-				)
-				(hide yes)
-			)
-		)
-		(property "Description" "Push button switch, normally open, two pins, 45° tilted"
-			(at 185.42 99.06 0)
-			(effects
-				(font
-					(size 1.27 1.27)
-				)
-				(hide yes)
-			)
-		)
-		(pin "1"
-		)
-		(pin "2"
-		)
-		(instances
-			(project "ortho-normal-keycap"
-				(path "/75ca063f-3e3a-4a56-b625-1bf464e147b8"
-					(reference "SW34")
-					(unit 1)
-				)
-			)
-		)
-	)
-	(symbol
-		(lib_id "ScottoKeebs:Placeholder_Keyswitch")
 		(at 215.9 99.06 0)
 		(unit 1)
@@
 			)
 		)
-		(property "Footprint" "eaglevlib-mx:SW_MX_1u"
+		(property "Footprint" "eaglevlib-mx:SW_MX_1.5u"
 			(at 185.42 81.28 0)
 			(effects
@@
 			)
 		)
-		(property "Footprint" "eaglevlib-mx:SW_MX_1u"
+		(property "Footprint" "eaglevlib-mx:SW_MX_CapsLock"
 			(at 185.42 99.06 0)
 			(effects
@@
 			)
 		)
-		(property "Footprint" "eaglevlib-mx:SW_MX_1u"
+		(property "Footprint" "eaglevlib-mx:SW_MX_1.25u"
 			(at 195.58 134.62 0)
 			(effects

Commit message: replace nRF52840 with nice!nano
Parts:
- removed U1: nRF52840_E73-2G4M08S1C, PCM_marbastlib-various:nRF52840_E73-2G4M08S1C, symbol PCM_marbastlib-various:nRF52840_E73-2G4M08S1C
- added U2: nice_nano, PCM_marbastlib-xp-promicroish:nice_nano_AH_USBup, symbol PCM_marbastlib-promicroish:nice_nano
- S23: renamed from S2; value MX_stab -> S2
- S33: renamed from S1; value MX_stab -> S1
Connections:
- net Col 0: now also U2.5 (P0.17)
- net Col 1: now also U2.6 (P0.20)
- net Col 2: now also U2.7 (P0.22)
- net Col 3: now also U2.8 (P0.24)
- net Col 4: now also U2.9 (P1.00)
- net Col 5: now also U2.10 (P0.11)
- net Row 0: now also U2.24 (P0.09-LF)
- net Row 1: now also U2.23 (P0.10-LF)
- net Row 2: now also U2.22 (P1.11-LF)
- net Row 3: now also U2.21 (P1.13-LF)
- net Row 4: now also U2.20 (P1.15-LF)
